Commit message: Chassis: the Waveshare UGV Rover, measured; and a plan for guarded verbs
PLAN-ros-alignment.md 3.20. The user chose the UGV Rover PT Jetson Orin
ROS2 Kit Acce (not yet ordered). Every copy of the chassis now carries its
numbers: 80 mm wheels, 1650 pulses/rev and a 0.172 m track (the stock
firmware's mainType 2, read from Waveshare's source) and a 253 x 231 mm
body -- sim, hardware backend, fake ESP32, URDF, controllers.yaml, nav2 and
robot/safety.py.

Measured on data, criteria written first: the body reaches all 13 rooms of
the furnished home (tests/chassis_fit.py, a C-space check on ground truth,
shown to catch a misfit first); the 3.18/3.19 safety sweeps pass unchanged;
the nav2 home tour is 8 of 9 on both chassis. Criterion 5 FAILS: 17
rule-based mission tests, because a direct-mode FORWARD verb is vetted once
and then drives a whole cell, parking the Rover where it cannot pivot. The
same gap lets the real car drive up to 10 cm past a wall under
`drive: direct` on either chassis -- recorded, not fixed.

PLAN-guarded-verbs.md is the plan for that fix (re-check direct-mode moves
every period, turns included, and make /stop end a hardware verb), saved
at the user's request with three decisions still open. Also: an offline
test that the xacro is well-formed XML, after a `--` in a comment stopped
the container from launching.

Co-Authored-By: Claude Opus 5.5 <noreply@anthropic.com>
Claude-Session: https://claude.ai/code/session_01CL2KVYsWCWnSRyLXtfm1uY

File: service/slam/src/picar_description/urdf/picar.urdf.xacro (robot description, xacro)
@@ -14,9 +14,13 @@
 <robot name="picar" xmlns:xacro="http://www.ros.org/wiki/xacro">
   <!-- ===================== every dimension ===================== -->
-  <xacro:property name="wheel_radius"      value="0.0325"/> <!-- [BOM] 65 mm wheels; = sim/mock_robot.py WHEEL_RADIUS_M -->
-  <xacro:property name="wheel_separation"  value="0.172"/>  <!-- [PLACEHOLDER] = sim/mock_robot.py TRACK_WIDTH_M, itself flagged -->
-  <xacro:property name="wheel_width"       value="0.026"/>  <!-- [PLACEHOLDER] -->
-  <xacro:property name="deck_length"       value="0.228"/>  <!-- [BOM] ~228 x 148 mm deck -->
-  <xacro:property name="deck_width"        value="0.148"/>  <!-- [BOM] -->
+  <!-- The Waveshare UGV Rover (PLAN-ros-alignment.md 3.20). Six wheels, four
+       driven, skid steer; modelled as one wheel a side, as a skid-steer
+       base usually is for diff_drive_controller; its larger EFFECTIVE track
+       is wheel_separation_multiplier, measured on the car. -->
+  <xacro:property name="wheel_radius"      value="0.040"/>  <!-- [BOM] 80 mm tyres, firmware mainType 2 WHEEL_D; = sim/mock_robot.py WHEEL_RADIUS_M -->
+  <xacro:property name="wheel_separation"  value="0.172"/>  <!-- [BOM] firmware mainType 2 TRACK_WIDTH; = sim/mock_robot.py TRACK_WIDTH_M -->
+  <xacro:property name="wheel_width"       value="0.0425"/> <!-- [BOM] 42.5 mm tyres -->
+  <xacro:property name="body_length"       value="0.253"/>  <!-- [BOM] outer, 253 x 231 mm: the FOOTPRINT nav2 and robot/safety.py use -->
+  <xacro:property name="body_width"        value="0.231"/>  <!-- [BOM] outer; the shell, not the wheels, sets the width -->
   <xacro:property name="deck_height"       value="0.040"/>  <!-- [PLACEHOLDER] chassis plate ~40 mm (CLAUDE.md Stage 0) -->
   <xacro:property name="axle_x"            value="0.0"/>    <!-- [PLACEHOLDER] drive axle under the deck centre -->
@@ -33,9 +37,9 @@
     <visual>
       <origin xyz="${-axle_x} 0 ${deck_height/2}"/>
-      <geometry><box size="${deck_length} ${deck_width} ${deck_height}"/></geometry>
+      <geometry><box size="${body_length} ${body_width} ${deck_height}"/></geometry>
     </visual>
     <collision>
       <origin xyz="${-axle_x} 0 ${deck_height/2}"/>
-      <geometry><box size="${deck_length} ${deck_width} ${deck_height}"/></geometry>
+      <geometry><box size="${body_length} ${body_width} ${deck_height}"/></geometry>
     </collision>
   </link>
@@ -49,10 +53,10 @@
   <joint name="front_bumper_joint" type="fixed">
     <parent link="base_link"/><child link="front_bumper"/>
-    <origin xyz="${deck_length/2 - axle_x} 0 0"/>
+    <origin xyz="${body_length/2 - axle_x} 0 0"/>
   </joint>
   <link name="rear_bumper"/>
   <joint name="rear_bumper_joint" type="fixed">
     <parent link="base_link"/><child link="rear_bumper"/>
-    <origin xyz="${-deck_length/2 - axle_x} 0 0"/>
+    <origin xyz="${-body_length/2 - axle_x} 0 0"/>
   </joint>
   <xacro:macro name="wheel" params="side y">

Commit message: 3.27: the Rover's CAD geometry, and the lidar 4 cm off-centre end to end
The xacro takes Waveshare's CAD (laser 4 cm ahead, pan axis 0.9 cm behind
the centre, lens 0.21 m up), pinned by tests/test_cad_geometry.py. The lidar
offset is one number -- LIDAR_X_M = laser_x = the sim's scan origin, a new
wall-linter entry (budget 10 -> 11) -- and every distance-to-chassis reader
moves returns into the body frame (scan_points_cm(); arrival too).

With safety still assuming a centred lidar, 177/2880 sweep runs ended under
18 cm and 56/120 close pivots touched; fixed, 0 and 0. PIVOT_MARGIN_CM
1.2 -> 1.3, moved after one guarded turn read 0.96 cm (rear corners now seen
from 4 cm farther), recorded in the plan. R3 criterion 4 now passes (1.89
deg at 1 m, was 4.59): strict xfail removed. SLAM maps at 100% precision;
final error 2.6-4.7 cm vs 1.5-3.6 control over four laps each.

Co-Authored-By: Claude Opus 5.5 <noreply@anthropic.com>
Claude-Session: https://claude.ai/code/session_01CL2KVYsWCWnSRyLXtfm1uY

File: service/slam/src/picar_description/urdf/picar.urdf.xacro (robot description, xacro)
@@ -23,10 +23,16 @@
   <xacro:property name="body_length"       value="0.253"/>  <!-- [BOM] outer, 253 x 231 mm: the FOOTPRINT nav2 and robot/safety.py use -->
   <xacro:property name="body_width"        value="0.231"/>  <!-- [BOM] outer; the shell, not the wheels, sets the width -->
+  <!-- [CAD] values are Waveshare's ugv_rover.urdf (ugv_ws @ f0b3ad9, BSD),
+       converted to these frames in PLAN-ros-alignment.md 3.27 and pinned by
+       tests/test_cad_geometry.py. CAD, not a tape measure: re-measure on
+       the car. -->
   <xacro:property name="deck_height"       value="0.040"/>  <!-- [PLACEHOLDER] chassis plate ~40 mm (CLAUDE.md Stage 0) -->
-  <xacro:property name="axle_x"            value="0.0"/>    <!-- [PLACEHOLDER] drive axle under the deck centre -->
-  <xacro:property name="laser_z"           value="0.100"/>  <!-- [PLACEHOLDER] lidar above base_link, deck centre -->
-  <xacro:property name="pan_x"             value="0.080"/>  <!-- [PLACEHOLDER] pan axis ahead of base_link -->
-  <xacro:property name="pan_z"             value="0.070"/>  <!-- [PLACEHOLDER] -->
-  <xacro:property name="camera_up"         value="0.0175"/> <!-- [PLACEHOLDER] lens above the pan joint: camera 0.12 m off the floor -->
+  <xacro:property name="axle_x"            value="0.0"/>    <!-- [CAD] driven wheels symmetric at +/-0.0855 m about the centre -->
+  <xacro:property name="laser_x"           value="0.040"/>  <!-- [CAD] lidar ahead of base_link; = robot/safety.py LIDAR_X_M and the sim's scan origin. The D500 is also mounted YAWED +90 deg (its zero faces left): not modelled, because the sim publishes the scan with zero ahead; a hardware-day item (3.27) -->
+  <xacro:property name="laser_z"           value="0.080"/>  <!-- [CAD] lidar 0.120 m off the floor -->
+  <xacro:property name="pan_x"             value="-0.009"/> <!-- [CAD] pan axis just BEHIND base_link -->
+  <xacro:property name="pan_z"             value="0.128"/>  <!-- [CAD] pan joint 0.168 m off the floor -->
+  <xacro:property name="camera_x"          value="0.048"/>  <!-- [CAD] lens ahead of the pan axis -->
+  <xacro:property name="camera_up"         value="0.042"/>  <!-- [CAD] lens above the pan joint: 0.210 m off the floor -->
   <xacro:property name="camera_pitch"      value="0.2618"/> <!-- [PLACEHOLDER] 15 deg down; the wedge is 10-20 deg, unmodelled -->
   <xacro:property name="pan_limit"         value="1.5708"/> <!-- [PLACEHOLDER] +/-90 deg; ST3215 can do more, the cable cannot -->
@@ -78,5 +84,5 @@
   <joint name="laser_joint" type="fixed">
     <parent link="base_link"/><child link="laser"/>
-    <origin xyz="${-axle_x} 0 ${laser_z}"/>
+    <origin xyz="${laser_x - axle_x} 0 ${laser_z}"/>
   </joint>
   <!-- The camera pans; bearings compose through this joint. -->
@@ -91,5 +97,5 @@
   <joint name="camera_joint" type="fixed">
     <parent link="pan_link"/><child link="camera_link"/>
-    <origin xyz="0 0 ${camera_up}" rpy="0 ${camera_pitch} 0"/>
+    <origin xyz="${camera_x} 0 ${camera_up}" rpy="0 ${camera_pitch} 0"/>
   </joint>
   <!-- REP-103's optical convention (z forward, x right, y down), for an
